File: pcb/esp-pogrammer.kicad_sch (KiCad schematic)
At the start: 31 parts, among them J1 USB_C_Receptacle_USB2.0, J2 TC2030-IDC, Q1 MMDT3904, Q2 MMDT3904, SW1 SW_SPDT, SW2 SW_Push, SW3 SW_Push, U1 CH340G, U2 AMS1117-3.3, Y1 12 MHz

Commit message: updates layout
Connections:
- net +3V3: no longer R5.1
- net 3.3V OUT: now also R5.1
Changed lines of the file:
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@@
+    )
+  )
+  (global_label "3.3V OUT" (shape input) (at 107.95 26.035 180) (fields_autoplaced)
+    (effects (font (size 1.27 1.27)) (justify right))
+    (property "Intersheet References" "${INTERSHEET_REFS}" (id 0) (at 96.8283 26.1144 0)
+      (effects (font (size 1.27 1.27)) (justify right) hide)
     )
   )
@@
     )
     (property "Datasheet" "" (id 3) (at 39.37 190.5 0)
-      (effects (font (size 1.27 1.27)) hide)
-    )
-    (pin "1")
-  )
-  (symbol (lib_id "power:+3.3V") (at 107.95 26.035 0) (unit 1)
-    (in_bom yes) (on_board yes) (fields_autoplaced)
-    (property "Reference" "#PWR0101" (id 0) (at 107.95 29.845 0)
-      (effects (font (size 1.27 1.27)) hide)
-    )
-    (property "Value" "+3.3V" (id 1) (at 107.95 20.701 0))
-    (property "Footprint" "" (id 2) (at 107.95 26.035 0)
-      (effects (font (size 1.27 1.27)) hide)
-    )
-    (property "Datasheet" "" (id 3) (at 107.95 26.035 0)
       (effects (font (size 1.27 1.27)) hide)
     )
@@
       (reference "#FLG0102") (unit 1) (value "PWR_FLAG") (footprint "")
     )
-    (path "/1a5f9495-1ac3-44fc-a7ee-ecec25e962fe"
-      (reference "#PWR0101") (unit 1) (value "+3.3V") (footprint "")
-    )
     (path "/15f0d612-18b7-4275-aeb7-cf595c193c23"

Commit message: added some filter caps, replaced local chip filter, replaced crystal caps, fixed switched power on reset, routed, rounded.
Parts:
- removed C5: 10uF, Capacitor_SMD:C_0603_1608Metric, symbol Device:C
- added C5: 0.1uF, Capacitor_SMD:C_0603_1608Metric, symbol pspice:CAP
- added C9: 10uF, Capacitor_SMD:C_0603_1608Metric, symbol pspice:CAP
- C1, C3: value 10uF -> 22pF
Connections:
- net +3V3: now also R5.1, C5.1, C9.1
- net 3.3V OUT: no longer R5.1
- net GND: now also C5.2, C9.2
Other:
- moved on the sheet: C8, D1, D2, D3, D4, R5, R6, R7, R8, R9, SW1, SW2

Commit message: fixed transistors. minor changes. ordered prototype 0.1.
Parts:
- Q1, Q2: value MMDT3904 -> S8050; footprint Package_TO_SOT_SMD:SOT-363_SC-70-6 -> Package_TO_SOT_SMD:SOT-23
Connections:
- net BOOT: now also Q2.3 (C3); no longer Q2.6 (C1)
- net DTR: now also Q2.2 (E2); no longer Q2.1 (E1)
- net RESET: now also Q1.3 (C3); no longer Q1.6 (C1)
- net RTS: now also Q1.2 (E2); no longer Q1.1 (E1)
- net at R4.2: now also Q2.1 (B1); no longer Q2.2 (B1)
- net at R3.2: now also Q1.1 (B1); no longer Q1.2 (B1)
